File: Electronics/EggbotWireless/EggbotWireless.sch (KiCad schematic (older format))
At the start: 59 parts, among them J1 BATT, J2 Conn_01x04_Female, J3 USB_B_Micro, J4 AVR-ISP-6, J5 Conn_01x03_Female, M1 Stepper_Motor_bipolar, M2 Stepper_Motor_bipolar, M3 Motor_Servo, Q1 FDD8447L, Q2 2N7002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

Commit message: use ft232rl for usb ic, better power handling
Parts:
- removed C12: 220uF, Capacitor_SMD:CP_Elec_10x10.5, symbol Device:CP
- removed U2: ATmega32A-AU, Package_QFP:TQFP-44_10x10mm_P0.8mm, symbol MCU_Microchip_ATmega:ATmega32A-AU
- removed U4: FS8205A, Package_SO:TSSOP-8_4.4x3mm_P0.65mm, symbol EggbotWireless-rescue:FS8205A-8205-Catfi-rescue
- removed U5: CP2102-GMR, Package_DFN_QFN:QFN-28-1EP_5x5mm_P0.5mm_EP3.35x3.35mm, symbol EggbotWireless-rescue:INTERFACE-CP2102-GMR(QFN28)-CP2102-GMR-Catfi-rescue
- added C16: 100nf, Capacitor_SMD:C_0805_2012Metric_Pad1.15x1.40mm_HandSolder, symbol EggbotWireless-rescue:C-Device-Catfi-rescue
- added D2: SK84, Diode_SMD:D_SMB_Handsoldering, symbol Device:D_Schottky
- added JP1, JP2, JP3: (no value), Jumper:SolderJumper-2_P1.3mm_Open_Pad1.0x1.5mm, symbol Jumper:SolderJumper_2_Open
- added Q3: AOD403, Package_TO_SOT_SMD:TO-252-2, symbol Device:Q_PMOS_GDS
- added U2: ATmega328P-AU, Package_QFP:TQFP-32_7x7mm_P0.8mm, symbol MCU_Microchip_ATmega:ATmega328P-AU
- added U4: DMG4800LSD, Package_SO:SO-8_3.9x4.9mm_P1.27mm, symbol DMG4800LSD:DMG4800LSD
- added U5: FT232RL, Package_SO:SSOP-28_5.3x10.2mm_P0.65mm, symbol Interface_USB:FT232RL
- C13: footprint Capacitor_SMD:CP_Elec_10x10.5 -> Capacitor_SMD:CP_Elec_8x10.5
- J1: footprint Connector_PinSocket_2.54mm:PinSocket_1x02_P2.54mm_Vertical -> Connector_PinHeader_2.54mm:PinHeader_1x02_P2.54mm_Vertical
- J2: footprint Connector_PinSocket_2.54mm:PinSocket_1x04_P2.54mm_Vertical -> Connector_PinHeader_2.54mm:PinHeader_1x04_P2.54mm_Vertical
- J5, M3: footprint Connector_PinSocket_2.54mm:PinSocket_1x03_P2.54mm_Vertical -> Connector_PinHeader_2.54mm:PinHeader_1x03_P2.54mm_Vertical
- M1, M2: value Stepper_Motor_bipolar -> (none); footprint Connector_PinSocket_2.54mm:PinSocket_1x04_P2.54mm_Vertical -> Connector_PinHeader_2.54mm:PinHeader_1x04_P2.54mm_Vertical
- R7: value 1K6 -> 2.2K
- SW1: value SW_SPDT -> (none)
Connections:
- net labels added: +5V, DIR1, DIR2, STEP1, STEP2, USBD+, USBD-
- wire segments 211 -> 220
Other:
- moved on the sheet: C1, C14, C15, C2, C3, C4, C5, C7, C8, J1, J2, J3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

Commit message: add uart pin header for esp12
Parts:
- added J6: Conn_01x05_Male, Connector_PinHeader_2.54mm:PinHeader_1x05_P2.54mm_Vertical, symbol Connector:Conn_01x05_Male
Changed lines of the file:
@@
 Text GLabel 7500 2200 2    50   Input ~ 0
 VBUS
-Text GLabel 8200 2900 2    50   Input ~ 0
-DTR_USB
-Text GLabel 8200 2500 2    50   Input ~ 0
-TXD_USB
-Text GLabel 8200 2600 2    50   Input ~ 0
-RXD_USB
-Text GLabel 8200 2700 2    50   Input ~ 0
-RTS_USB
 $Comp
 L Interface_USB:FT232RL U5
@@
 Wire Wire Line
 	8800 2300 8800 2100
+Text GLabel 8200 2700 2    50   Input ~ 0
+RTS_USB
+Text GLabel 8200 2600 2    50   Input ~ 0
+RXD_USB
+Text GLabel 8200 2500 2    50   Input ~ 0
+TXD_USB
+Text GLabel 8200 2900 2    50   Input ~ 0
+DTR_USB
+Text GLabel 5600 2200 2    50   Input ~ 0
+TXD_USB
+$Comp
+L Connector:Conn_01x05_Male J6
+U 1 1 5D0DB384
+P 5400 2400
+F 0 "J6" H 5508 2781 50  0000 C CNN
+F 1 "Conn_01x05_Male" H 5508 2690 50  0000 C CNN
+F 2 "Connector_PinHeader_2.54mm:PinHeader_1x05_P2.54mm_Vertical" H 5400 2400 50  0001 C CNN
+F 3 "~" H 5400 2400 50  0001 C CNN
+	1    5400 2400
+	1    0    0    -1
+$EndComp
+Text GLabel 5600 2300 2    50   Input ~ 0
+RXD_USB
+Text GLabel 5600 2400 2    50   Input ~ 0
+RTS_USB
+Text GLabel 5600 2500 2    50   Input ~ 0
+DTR_USB
+$Comp
+L EggbotWireless-rescue:GND-power-Catfi-rescue #PWR0147
+U 1 1 5D0DD546
+P 5600 2600
+F 0 "#PWR0147" H 5600 2350 50  0001 C CNN
+F 1 "GND" H 5605 2427 50  0000 C CNN
+F 2 "" H 5600 2600 50  0001 C CNN
+F 3 "" H 5600 2600 50  0001 C CNN
+	1    5600 2600
+	1    0    0    -1
+$EndComp
 $EndSCHEMATC

Commit message: pcb v1.1 proto
Parts:
- added R20: 100K, Resistor_SMD:R_0805_2012Metric_Pad1.15x1.40mm_HandSolder, symbol EggbotWireless-rescue:R-Device-Catfi-rescue
- R6: value 10K -> 100K
Connections:
- wire segments 220 -> 224
Changed lines of the file:
@@
 	-1   0    0    1
 $EndComp
-Wire Wire Line
-	1000 1250 1000 1350
 $Comp
 L EggbotWireless-rescue:R-Device-Catfi-rescue R1
@@
 F 3 "" H 1550 4050 50  0001 C CNN
 	1    1550 4050
-	1    0    0    -1
+	0    -1   -1   0
 $EndComp
 $Comp
@@
 	1    0    0    -1
 $EndComp
-Text GLabel 1700 7000 0    50   Input ~ 0
+Text GLabel 2900 6600 2    50   Input ~ 0
 12V_SWITCH
-Text GLabel 8400 5850 1    50   Input ~ 0
+Text GLabel 8200 5850 1    50   Input ~ 0
 12V_SWITCH
 $Comp
@@
 L EggbotWireless-rescue:GND-power-Catfi-rescue #PWR0152
 U 1 1 5CFAA2C4
-P 8700 6050
-F 0 "#PWR0152" H 8700 5800 50  0001 C CNN
-F 1 "GND" H 8705 5877 50  0000 C CNN
-F 2 "" H 8700 6050 50  0001 C CNN
-F 3 "" H 8700 6050 50  0001 C CNN
-	1    8700 6050
-	1    0    0    -1
+P 8700 6200
+F 0 "#PWR0152" H 8700 5950 50  0001 C CNN
+F 1 "GND" H 8705 6027 50  0000 C CNN
+F 2 "" H 8700 6200 50  0001 C CNN
+F 3 "" H 8700 6200 50  0001 C CNN
+	1    8700 6200
+	0    -1   -1   0
 $EndComp
 $Comp
@@
 P 10050 1300
 F 0 "R6" V 9843 1300 50  0000 C CNN
-F 1 "10K" V 9934 1300 50  0000 C CNN
+F 1 "100K" V 9934 1300 50  0000 C CNN
 F 2 "Resistor_SMD:R_0805_2012Metric_Pad1.15x1.40mm_HandSolder" V 9980 1300 50  0001 C CNN
 F 3 "~" H 10050 1300 50  0001 C CNN
@@
 	1    0    0    -1
 $EndComp
+$Comp
+L EggbotWireless-rescue:R-Device-Catfi-rescue R20
+U 1 1 5D171129
+P 8300 6000
+F 0 "R20" V 8093 6000 50  0000 C CNN
+F 1 "100K" V 8184 6000 50  0000 C CNN
+F 2 "Resistor_SMD:R_0805_2012Metric_Pad1.15x1.40mm_HandSolder" V 8230 6000 50  0001 C CNN
+F 3 "~" H 8300 6000 50  0001 C CNN
+	1    8300 6000
+	-1   0    0    1
+$EndComp
+Wire Wire Line
+	8200 5850 8300 5850
+Wire Wire Line
+	8300 5850 8400 5850
+Connection ~ 8300 5850
+Wire Wire Line
+	8700 6200 8700 6050
+Wire Wire Line
+	8300 6150 8300 6200
+Wire Wire Line
+	8300 6200 8700 6200
+Connection ~ 8700 6200
 $EndSCHEMATC

Commit message: use nodemcu reset circuit
Parts:
- removed J2: Conn_01x04_Female, Connector_PinHeader_2.54mm:PinHeader_1x04_P2.54mm_Vertical, symbol EggbotWireless-rescue:Conn_01x04_Female-Connector-Catfi-rescue
- added C12: 220uF, Capacitor_SMD:CP_Elec_8x10.5, symbol Device:CP
- added D3: LED, Diode_SMD:D_0805_2012Metric_Pad1.15x1.40mm_HandSolder, symbol Device:LED
- added J2: Conn_01x03_Male, Connector_PinHeader_2.54mm:PinHeader_1x03_P2.54mm_Vertical, symbol Connector:Conn_01x03_Male
- added Q4: 2N7002, Package_TO_SOT_SMD:SOT-23, symbol Transistor_FET:2N7002
- added Q5, Q6: S8050, Package_TO_SOT_SMD:SOT-23, symbol Device:Q_NPN_BEC
- added R21: 330, Resistor_SMD:R_0805_2012Metric_Pad1.15x1.40mm_HandSolder, symbol EggbotWireless-rescue:R-Device-Catfi-rescue
- added R22: 100K, Resistor_SMD:R_0805_2012Metric_Pad1.15x1.40mm_HandSolder, symbol EggbotWireless-rescue:R-Device-Catfi-rescue
- added R23: 10K, Resistor_SMD:R_0805_2012Metric_Pad1.15x1.40mm_HandSolder, symbol EggbotWireless-rescue:R-Device-Catfi-rescue
- added R24, R25: 12K, Resistor_SMD:R_0805_2012Metric_Pad1.15x1.40mm_HandSolder, symbol EggbotWireless-rescue:R-Device-Catfi-rescue
Connections:
- net labels added: CHEN, ESPRST, GPIO0, PWREN, SLEEP
- net labels removed: +BATT
- wire segments 224 -> 231
Other:
- moved on the sheet: C16, C5

Commit message: fix issue with ft232rl being powered with rx/tx board v1.1b
Connections:
- net +5V: now also C16.2, U5.20 (VCC)
- net VBUS: no longer C16.2, U5.20 (VCC)
Changed lines of the file:
@@
 	0    -1   -1   0
 $EndComp
-Text GLabel 7500 2200 2    50   Input ~ 0
-VBUS
 $Comp
 L Interface_USB:FT232RL U5
@@
 	1    0    0    -1
 $EndComp
+$Comp
+L power:+5V #PWR?
+U 1 1 5D283EF7
+P 7500 2200
+F 0 "#PWR?" H 7500 2050 50  0001 C CNN
+F 1 "+5V" H 7515 2373 50  0000 C CNN
+F 2 "" H 7500 2200 50  0001 C CNN
+F 3 "" H 7500 2200 50  0001 C CNN
+	1    7500 2200
+	0    1    1    0
+$EndComp
+Connection ~ 7500 2200
 $EndSCHEMATC

Commit message: board v1.2 use p-mosfet for charge enable/disable use sleep instead of pwren connect battery to esp adc via voltage divider
Parts:
- removed Q4: 2N7002, Package_TO_SOT_SMD:SOT-23, symbol Transistor_FET:2N7002
- removed R23: 10K, Resistor_SMD:R_0805_2012Metric_Pad1.15x1.40mm_HandSolder, symbol EggbotWireless-rescue:R-Device-Catfi-rescue
- added Q4: IRLML6402, Package_TO_SOT_SMD:SOT-23, symbol Transistor_FET:IRLML6402
- added R26: 12K, Resistor_SMD:R_0805_2012Metric_Pad1.15x1.40mm_HandSolder, symbol EggbotWireless-rescue:R-Device-Catfi-rescue
- added R27: 3K, Resistor_SMD:R_0805_2012Metric_Pad1.15x1.40mm_HandSolder, symbol EggbotWireless-rescue:R-Device-Catfi-rescue
Connections:
- net CHEN: now also Q4.1 (G)
- net GND: now also Q4.3 (D), R27.2
- net SLEEP: now also U7.19 (GPIO4)
- net BATT: now reaches J1.2 (Pin_2), Q3.2 (D), R2.2, U6.3 (BAT)
- net BATT: now also R26.1
- net at R7.2: now also Q4.2 (S)
- net at U7.2 (ADC): now also R26.2, R27.1
- net PWREN: no longer names the net of U5.14 (CBUS3)
- net PWREN: no longer U7.19 (GPIO4)
Other:
- moved on the sheet: J6

Commit message: fix some power issues
Parts:
- removed JP1, JP2, JP3: (no value), Jumper:SolderJumper-2_P1.3mm_Open_Pad1.0x1.5mm, symbol Jumper:SolderJumper_2_Open
- removed Q3: AOD403, Package_TO_SOT_SMD:TO-252-2, symbol Device:Q_PMOS_GDS
- added C17: 10uF, Capacitor_SMD:C_0805_2012Metric_Pad1.15x1.40mm_HandSolder, symbol Device:C
- added D4: SSB43L, Diode_SMD:D_SMB_Handsoldering, symbol Device:D_Schottky
- added JP1, JP2, JP3: SolderJumper_2_Bridged, Jumper:SolderJumper-2_P1.3mm_Bridged_Pad1.0x1.5mm, symbol Jumper:SolderJumper_2_Bridged
- added Q3: IRLML6402, Package_TO_SOT_SMD:SOT-23, symbol Transistor_FET:IRLML6402
- D1: value SK24 -> SSB43L
- D2: value SK84 -> SSB43L
- Q1: value FDD8447L -> FDD8800
- R15: value 0.006 -> 0.008
- R16: value 9.1K -> 8.45K
- R20, R22, R6: value 100K -> 10K
Connections:
- net +3V3: now also JP1.1 (A), JP2.1 (A), JP3.1 (A)
- net +5V: now also C17.1
- net BATT: now also D4.2 (A)
- net GND: now also C17.2
- net VBUS: now also Q3.1 (G)
- net at A1.10 (M0), A2.10 (M0): now also JP3.2 (B)
- net at A1.11 (M1), A2.11 (M1): now also JP2.2 (B)
- net at A1.12 (M2), A2.12 (M2): now also JP1.2 (B)
- net at D2.1 (K), SW1.2 (B): now also Q3.3 (D)
- new net: D4.1 (K), Q3.2 (S)
Other:
- moved on the sheet: SW1
Changed lines of the file:
@@
 P 9950 4450
 F 0 "D1" H 9950 4234 50  0000 C CNN
-F 1 "SK24" H 9950 4325 50  0000 C CNN
+F 1 "SSB43L" H 9950 4325 50  0000 C CNN
 F 2 "Diode_SMD:D_SMB_Handsoldering" H 9950 4450 50  0001 C CNN
 F 3 "~" H 9950 4450 50  0001 C CNN
@@
 	9050 4450 9300 4450
 Wire Wire Line
-	9050 3850 9300 3850
-Wire Wire Line
 	9600 4450 9700 4450
 Wire Wire Line
@@
 P 9700 5350
 F 0 "R15" H 9770 5396 50  0000 L CNN
-F 1 "0.006" H 9770 5305 50  0000 L CNN
+F 1 "0.008" H 9770 5305 50  0000 L CNN
 F 2 "Resistor_SMD:R_1206_3216Metric_Pad1.42x1.75mm_HandSolder" V 9630 5350 50  0001 C CNN
 F 3 "~" H 9700 5350 50  0001 C CNN
@@
 P 10200 5400
 F 0 "R16" H 10270 5446 50  0000 L CNN
-F 1 "9.1K" H 10270 5355 50  0000 L CNN
+F 1 "8.45K" H 10270 5355 50  0000 L CNN
 F 2 "Resistor_SMD:R_0805_2012Metric_Pad1.15x1.40mm_HandSolder" V 10130 5400 50  0001 C CNN
 F 3 "~" H 10200 5400 50  0001 C CNN
@@
 	1    0    0    -1
 $EndComp
-Connection ~ 9300 3850
 $Comp
 L EggbotWireless-rescue:GND-power-Catfi-rescue #PWR0136
 U 1 1 5D0FBB70
-P 9300 4150
-F 0 "#PWR0136" H 9300 3900 50  0001 C CNN
-F 1 "GND" H 9305 3977 50  0000 C CNN
-F 2 "" H 9300 4150 50  0001 C CNN
-F 3 "" H 9300 4150 50  0001 C CNN
-	1    9300 4150
+P 9300 4200
+F 0 "#PWR0136" H 9300 3950 50  0001 C CNN
+F 1 "GND" H 9305 4027 50  0000 C CNN
+F 2 "" H 9300 4200 50  0001 C CNN
+F 3 "" H 9300 4200 50  0001 C CNN
+	1    9300 4200
 	1    0    0    -1
 $EndComp
@@
 	4500 4150 4550 4150
 Wire Wire Line
-	4400 4350 4400 4250
-Wire Wire Line
 	4400 4250 4550 4250
 Wire Wire Line
-	4400 4350 4400 6100
-Wire Wire Line
 	4400 6100 4600 6100
-Connection ~ 4400 4350
 Wire Wire Line
 	4350 4550 4350 6200
@@
 Wire Wire Line
 	4450 4350 4550 4350
-Connection ~ 4350 4550
 $Comp
 L power:+3.3V #PWR0146
@@
 Wire Wire Line
 	4100 4150 4100 4350
-Connection ~ 4150 4150
 Wire Wire Line
 	4100 4350 4050 4350
 Wire Wire Line
 	4050 4350 4050 4550
-Connection ~ 4100 4350
-$Comp
-L Jumper:SolderJumper_2_Open JP3
-U 1 1 5D1FD66D
-P 4300 4150
-F 0 "JP3" H 4300 4250 50  0000 C CNN
-F 1 " " H 4300 4264 50  0000 C CNN
-F 2 "Jumper:SolderJumper-2_P1.3mm_Open_Pad1.0x1.5mm" H 4300 4150 50  0001 C CNN
-F 3 "~" H 4300 4150 50  0001 C CNN
-	1    4300 4150
-	1    0    0    -1
-$EndComp
-$Comp
-L Jumper:SolderJumper_2_Open JP2
-U 1 1 5D2160D7
-P 4250 4350
-F 0 "JP2" H 4250 4450 50  0000 C CNN
-F 1 " " H 4250 4464 50  0000 C CNN
-F 2 "Jumper:SolderJumper-2_P1.3mm_Open_Pad1.0x1.5mm" H 4250 4350 50  0001 C CNN
-F 3 "~" H 4250 4350 50  0001 C CNN
-	1    4250 4350
-	1    0    0    -1
-$EndComp
-$Comp
-L Jumper:SolderJumper_2_Open JP1
-U 1 1 5D2166DA
-P 4200 4550
-F 0 "JP1" H 4200 4650 50  0000 C CNN
-F 1 " " H 4200 4664 50  0000 C CNN
-F 2 "Jumper:SolderJumper-2_P1.3mm_Open_Pad1.0x1.5mm" H 4200 4550 50  0001 C CNN
-F 3 "~" H 4200 4550 50  0001 C CNN
-	1    4200 4550
-	1    0    0    -1
-$EndComp
 $Comp
 L power:+3.3V #PWR0138
@@
 	2050 800  2050 900
 Wire Wire Line
-	9300 3850 9300 3800
-Wire Wire Line
 	2200 5700 2300 5700
 Connection ~ 2200 5700
@@
 P 9600 4750
 F 0 "Q1" H 9806 4796 50  0000 L CNN
-F 1 "FDD8447L" H 9806 4705 50  0000 L CNN
+F 1 "FDD8800" H 9806 4705 50  0000 L CNN
 F 2 "Package_TO_SOT_SMD:TO-252-2" H 9800 4850 50  0001 C CNN
 F 3 "~" H 9600 4750 50  0001 C CNN
@@
 Wire Wire Line
 	7650 1000 7500 1000
-Connection ~ 7650 650
 Text GLabel 9900 1100 0    50   Input ~ 0
 VBUS
 Wire Wire Line
 	9900 1100 9900 1950
-Wire Wire Line
-	10450 1400 10450 1950
 $Comp
 L EggbotWireless-rescue:GND-power-Catfi-rescue #PWR0123
@@
 P 10050 1300
 F 0 "R6" V 9843 1300 50  0000 C CNN
-F 1 "100K" V 9934 1300 50  0000 C CNN
+F 1 "10K" V 9934 1300 50  0000 C CNN
 F 2 "Resistor_SMD:R_0805_2012Metric_Pad1.15x1.40mm_HandSolder" V 9980 1300 50  0001 C CNN
 F 3 "~" H 10050 1300 50  0001 C CNN
@@
 P 10150 1950
 F 0 "D2" H 10150 1734 50  0000 C CNN
-F 1 "SK84" H 10150 1825 50  0000 C CNN
+F 1 "SSB43L" H 10150 1825 50  0000 C CNN
 F 2 "Diode_SMD:D_SMB_Handsoldering" H 10150 1950 50  0001 C CNN
 F 3 "~" H 10150 1950 50  0001 C CNN
@@
 L Switch:SW_SPDT SW1
 U 1 1 5CEB7C0D
-P 10650 1400
-F 0 "SW1" H 10650 1550 50  0000 C CNN
-F 1 " " H 10650 1594 50  0000 C CNN
-F 2 "Button_Switch_THT:SW_CuK_OS102011MA1QN1_SPDT_Angled" H 10650 1400 50  0001 C CNN
-F 3 "~" H 10650 1400 50  0001 C CNN
-	1    10650 1400
-	1    0    0    -1
-$EndComp
-Connection ~ 10450 1400
+P 10750 1400
+F 0 "SW1" H 10750 1550 50  0000 C CNN
+F 1 " " H 10750 1594 50  0000 C CNN
+F 2 "Button_Switch_THT:SW_CuK_OS102011MA1QN1_SPDT_Angled" H 10750 1400 50  0001 C CNN
+F 3 "~" H 10750 1400 50  0001 C CNN
+	1    10750 1400
+	1    0    0    -1
+$EndComp
 $Comp
 L power:+5V #PWR0130
 U 1 1 5D7ABED4
-P 10850 1300
-F 0 "#PWR0130" H 10850 1150 50  0001 C CNN
-F 1 "+5V" H 10865 1473 50  0000 C CNN
-F 2 "" H 10850 1300 50  0001 C CNN
-F 3 "" H 10850 1300 50  0001 C CNN
-	1    10850 1300
-	1    0    0    -1
-$EndComp
-Wire Wire Line
-	7650 650  10350 650
+P 10950 1300
+F 0 "#PWR0130" H 10950 1150 50  0001 C CNN
+F 1 "+5V" H 10965 1473 50  0000 C CNN
+F 2 "" H 10950 1300 50  0001 C CNN
+F 3 "" H 10950 1300 50  0001 C CNN
+	1    10950 1300
+	1    0    0    -1
+$EndComp
 Wire Wire Line
 	10350 650  10350 900
 Wire Wire Line
-	10450 1950 10300 1950
-Wire Wire Line
 	10000 1950 9900 1950
-Connection ~ 10050 1100
-$Comp
-L Device:Q_PMOS_GDS Q3
-U 1 1 5D797440
-P 10250 1100
-F 0 "Q3" H 10456 1146 50  0000 L CNN
-F 1 "AOD403" H 10456 1055 50  0000 L CNN
-F 2 "Package_TO_SOT_SMD:TO-252-2" H 10450 1200 50  0001 C CNN
-F 3 "~" H 10250 1100 50  0001 C CNN
-	1    10250 1100
-	1    0    0    -1
-$EndComp
 $Comp
 L DMG4800LSD:DMG4800LSD U4
@@
 Text GLabel 8200 2900 2    50   Input ~ 0
 DTR_USB
-$Comp
-L EggbotWireless-rescue:R-Device-Catfi-rescue R20
-U 1 1 5D171129
-P 8300 6000
-F 0 "R20" V 8093 6000 50  0000 C CNN
-F 1 "100K" V 8184 6000 50  0000 C CNN
-F 2 "Resistor_SMD:R_0805_2012Metric_Pad1.15x1.40mm_HandSolder" V 8230 6000 50  0001 C CNN
-F 3 "~" H 8300 6000 50  0001 C CNN
-	1    8300 6000
-	-1   0    0    1
-$EndComp
 Wire Wire Line
 	8200 5850 8300 5850
@@
 P 5900 1800
 F 0 "R22" V 5693 1800 50  0000 C CNN
-F 1 "100K" V 5784 1800 50  0000 C CNN
+F 1 "10K" V 5784 1800 50  0000 C CNN
 F 2 "Resistor_SMD:R_0805_2012Metric_Pad1.15x1.40mm_HandSolder" V 5830 1800 50  0001 C CNN
 F 3 "~" H 5900 1800 50  0001 C CNN
@@
 Text GLabel 2900 6500 2    50   Input ~ 0
 SLEEP
+$Comp
+L EggbotWireless-rescue:R-Device-Catfi-rescue R20
+U 1 1 5D171129
+P 8300 6000
+F 0 "R20" V 8093 6000 50  0000 C CNN
+F 1 "10K" V 8184 6000 50  0000 C CNN
+F 2 "Resistor_SMD:R_0805_2012Metric_Pad1.15x1.40mm_HandSolder" V 8230 6000 50  0001 C CNN
+F 3 "~" H 8300 6000 50  0001 C CNN
+	1    8300 6000
+	-1   0    0    1
+$EndComp
+$Comp
+L Device:D_Schottky D4
+U 1 1 5D32EDF7
+P 10200 650
+F 0 "D4" H 10200 434 50  0000 C CNN
+F 1 "SSB43L" H 10200 525 50  0000 C CNN
+F 2 "Diode_SMD:D_SMB_Handsoldering" H 10200 650 50  0001 C CNN
+F 3 "~" H 10200 650 50  0001 C CNN
+	1    10200 650
+	-1   0    0    -1
+$EndComp
+Wire Wire Line
+	10050 650  7650 650
+Connection ~ 7650 650
+Wire Wire Line
+	9300 4200 9300 4150
+Wire Wire Line
+	9300 3850 9300 3800
+Connection ~ 9300 3850
+Wire Wire Line
+	9050 3850 9300 3850
+$Comp
+L Device:C C17
+U 1 1 5D338D3C
+P 9700 4000
+F 0 "C17" H 9815 4046 50  0000 L CNN
+F 1 "10uF" H 9815 3955 50  0000 L CNN
+F 2 "Capacitor_SMD:C_0805_2012Metric_Pad1.15x1.40mm_HandSolder" H 9738 3850 50  0001 C CNN
+F 3 "~" H 9700 4000 50  0001 C CNN
+	1    9700 4000
+	1    0    0    -1
+$EndComp
+Wire Wire Line
+	9300 3850 9700 3850
+Wire Wire Line
+	9700 4150 9300 4150
+Connection ~ 9300 4150
+$Comp
+L Transistor_FET:IRLML6402 Q3
+U 1 1 5D2DC610
+P 10250 1100
+F 0 "Q3" H 10456 1054 50  0000 L CNN
+F 1 "IRLML6402" H 10456 1145 50  0000 L CNN
+F 2 "Package_TO_SOT_SMD:SOT-23" H 10450 1025 50  0001 L CIN
+F 3 "https://www.infineon.com/dgdl/irlml6402pbf.pdf?fileId=5546d462533600a401535668d5c2263c" H 10250 1100 50  0001 L CNN
+	1    10250 1100
+	1    0    0    1
+$EndComp
+Connection ~ 10050 1100
+Wire Wire Line
+	10300 1950 10450 1950
+Wire Wire Line
+	10450 1950 10450 1400
+Connection ~ 10450 1400
+Wire Wire Line
+	10450 1400 10550 1400
+$Comp
+L Jumper:SolderJumper_2_Bridged JP3
+U 1 1 5D3CD55E
+P 4300 4150
+F 0 "JP3" H 4300 4355 50  0000 C CNN
+F 1 "SolderJumper_2_Bridged" H 4300 4264 50  0000 C CNN
+F 2 "Jumper:SolderJumper-2_P1.3mm_Bridged_Pad1.0x1.5mm" H 4300 4150 50  0001 C CNN
+F 3 "~" H 4300 4150 50  0001 C CNN
+	1    4300 4150
+	1    0    0    -1
+$EndComp
+$Comp
+L Jumper:SolderJumper_2_Bridged JP2
+U 1 1 5D3CED16
+P 4250 4350
+F 0 "JP2" H 4250 4555 50  0000 C CNN
+F 1 "SolderJumper_2_Bridged" H 4250 4464 50  0000 C CNN
+F 2 "Jumper:SolderJumper-2_P1.3mm_Bridged_Pad1.0x1.5mm" H 4250 4350 50  0001 C CNN
+F 3 "~" H 4250 4350 50  0001 C CNN
+	1    4250 4350
+	1    0    0    -1
+$EndComp
+$Comp
+L Jumper:SolderJumper_2_Bridged JP1
+U 1 1 5D3CF16C
+P 4200 4550
+F 0 "JP1" H 4200 4755 50  0000 C CNN
+F 1 "SolderJumper_2_Bridged" H 4200 4664 50  0000 C CNN
+F 2 "Jumper:SolderJumper-2_P1.3mm_Bridged_Pad1.0x1.5mm" H 4200 4550 50  0001 C CNN
+F 3 "~" H 4200 4550 50  0001 C CNN
+	1    4200 4550
+	1    0    0    -1
+$EndComp
+Wire Wire Line
+	4400 4250 4400 4350
+Connection ~ 4150 4150
+Connection ~ 4100 4350
+Connection ~ 4400 4350
+Wire Wire Line
+	4400 4350 4400 6100
+Connection ~ 4350 4550
 $EndSCHEMATC
