File: Electronics/EggbotWireless/EggbotWireless.sch (KiCad schematic (older format))
At the start: 79 parts, among them J1 BATT, J2 Conn_01x03_Male, J3 USB_B_Micro, J4 AVR-ISP-6, J5 Conn_01x03_Female, J6 Conn_01x05_Male, M1 , M2 , M3 Motor_Servo, Q1 FDD8800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

Commit message: board v1.3
Parts:
- A1, A2: symbol Driver_Motor:Pololu_Breakout_DRV8825 -> EggbotWireless-rescue:Pololu_Breakout_DRV8825-Driver_Motor
- C12, C13: symbol Device:CP -> EggbotWireless-rescue:CP-Device
- C17, C2, C5: symbol Device:C -> EggbotWireless-rescue:C-Device
- D1, D2, D4: symbol Device:D_Schottky -> EggbotWireless-rescue:D_Schottky-Device
- D3: symbol Device:LED -> EggbotWireless-rescue:LED-Device
- J2: symbol Connector:Conn_01x03_Male -> EggbotWireless-rescue:Conn_01x03_Male-Connector
- J4: symbol Connector:AVR-ISP-6 -> EggbotWireless-rescue:AVR-ISP-6-Connector
- J5: symbol Connector:Conn_01x03_Female -> EggbotWireless-rescue:Conn_01x03_Female-Connector
- J6: symbol Connector:Conn_01x05_Male -> EggbotWireless-rescue:Conn_01x05_Male-Connector
- JP1, JP2, JP3: symbol Jumper:SolderJumper_2_Bridged -> EggbotWireless-rescue:SolderJumper_2_Bridged-Jumper
- L1, L2: symbol Device:L -> EggbotWireless-rescue:L-Device
- M1, M2: symbol Motor:Stepper_Motor_bipolar -> EggbotWireless-rescue:Stepper_Motor_bipolar-Motor
- M3: symbol Motor:Motor_Servo -> EggbotWireless-rescue:Motor_Servo-Motor
- Q1: symbol Device:Q_NMOS_GDS -> EggbotWireless-rescue:Q_NMOS_GDS-Device
- Q2: symbol Transistor_FET:2N7002 -> EggbotWireless-rescue:2N7002-Transistor_FET
- Q3, Q4: symbol Transistor_FET:IRLML6402 -> EggbotWireless-rescue:IRLML6402-Transistor_FET
- Q5, Q6: symbol Device:Q_NPN_BEC -> EggbotWireless-rescue:Q_NPN_BEC-Device
- R13, R14, R15, R16, R19, R4, R5: symbol Device:R -> EggbotWireless-rescue:R-Device
- SW1: symbol Switch:SW_SPDT -> EggbotWireless-rescue:SW_SPDT-Switch
- U1: symbol Regulator_Switching:TPS62203DBV -> EggbotWireless-rescue:TPS62203DBV-Regulator_Switching
- U2: symbol MCU_Microchip_ATmega:ATmega328P-AU -> EggbotWireless-rescue:ATmega328P-AU-MCU_Microchip_ATmega
- U5: symbol Interface_USB:FT232RL -> EggbotWireless-rescue:FT232RL-Interface_USB
- Y1: symbol Device:Crystal -> EggbotWireless-rescue:Crystal-Device
Changed lines of the file:
@@
 $EndDescr
 $Comp
-L Device:L L2
+L EggbotWireless-rescue:L-Device L2
 U 1 1 5CE6FFE2
 P 10150 2650
@@
 $EndComp
 $Comp
-L Device:C C5
+L EggbotWireless-rescue:C-Device C5
 U 1 1 5CE79D1A
 P 10900 2800
@@
 $EndComp
 $Comp
-L Device:C C2
+L EggbotWireless-rescue:C-Device C2
 U 1 1 5CE7AF72
 P 9100 2900
@@
 	9350 3050 9650 3050
 $Comp
-L Regulator_Switching:TPS62203DBV U1
+L EggbotWireless-rescue:TPS62203DBV-Regulator_Switching U1
 U 1 1 5CE8E5BF
 P 9650 2850
@@
 	9950 2850 10350 2850
 $Comp
-L Device:D_Schottky D1
+L EggbotWireless-rescue:D_Schottky-Device D1
 U 1 1 5D005B12
 P 9950 4450
@@
 	1550 750  1550 800
 $Comp
-L power:+3.3V #PWR0107
+L EggbotWireless-rescue:+3.3V-power #PWR0107
 U 1 1 5CEB7CB7
 P 1550 750
@@
 $EndComp
 $Comp
-L Device:Crystal Y1
+L EggbotWireless-rescue:Crystal-Device Y1
 U 1 1 5CED63CD
 P 2700 1500
@@
 Connection ~ 2700 1050
 $Comp
-L power:+3.3V #PWR0129
+L EggbotWireless-rescue:+3.3V-power #PWR0129
 U 1 1 5D0C7E91
 P 2300 5700
@@
 	9050 3850 9050 4450
 $Comp
-L Device:L L1
+L EggbotWireless-rescue:L-Device L1
 U 1 1 5CEC224D
 P 9450 4450
@@
 	9400 4750 9050 4750
 $Comp
-L Device:R R15
+L EggbotWireless-rescue:R-Device R15
 U 1 1 5CEF81B9
 P 9700 5350
@@
 	9700 5200 9700 5100
 $Comp
-L Device:R R14
+L EggbotWireless-rescue:R-Device R14
 U 1 1 5CF00015
 P 9500 5100
@@
 Connection ~ 9300 5100
 $Comp
-L Device:CP C13
+L EggbotWireless-rescue:CP-Device C13
 U 1 1 5CF5EC34
 P 10400 4600
@@
 Connection ~ 8600 5050
 $Comp
-L Device:R R16
+L EggbotWireless-rescue:R-Device R16
 U 1 1 5CF6C873
 P 10200 5400
@@
 $EndComp
 $Comp
-L Device:R R5
+L EggbotWireless-rescue:R-Device R5
 U 1 1 5CF6CC3B
 P 7850 5150
@@
 $EndComp
 $Comp
-L Device:R R4
+L EggbotWireless-rescue:R-Device R4
 U 1 1 5CFEC7EA
 P 7500 5150
@@
 	7850 5350 7850 5300
 $Comp
-L Device:R R13
+L EggbotWireless-rescue:R-Device R13
 U 1 1 5D0DA168
 P 9100 5350
@@
 $EndComp
 $Comp
-L power:+3.3V #PWR0127
+L EggbotWireless-rescue:+3.3V-power #PWR0127
 U 1 1 5D03EF52
 P 3650 3150
@@
 $EndComp
 $Comp
-L Connector:AVR-ISP-6 J4
+L EggbotWireless-rescue:AVR-ISP-6-Connector J4
 U 1 1 5D029176
 P 3550 2650
@@
 $EndComp
 $Comp
-L Connector:Conn_01x03_Female J5
+L EggbotWireless-rescue:Conn_01x03_Female-Connector J5
 U 1 1 5CF7E398
 P 2850 3150
@@
 	5650 5900 5400 5900
 $Comp
-L power:+12V #PWR0142
+L EggbotWireless-rescue:+12V-power #PWR0142
 U 1 1 5CF0714E
 P 5000 5000
@@
 $EndComp
 $Comp
-L power:+12V #PWR0143
+L EggbotWireless-rescue:+12V-power #PWR0143
 U 1 1 5CF093C7
 P 4950 3150
@@
 Connection ~ 5000 4550
 $Comp
-L power:+3.3V #PWR0148
+L EggbotWireless-rescue:+3.3V-power #PWR0148
 U 1 1 5CF94114
 P 4600 5300
@@
 	4600 5300 4600 5400
 $Comp
-L power:+3.3V #PWR0149
+L EggbotWireless-rescue:+3.3V-power #PWR0149
 U 1 1 5CFA006C
 P 4550 3450
@@
 	4550 3450 4550 3550
 $Comp
-L Motor:Motor_Servo M3
+L EggbotWireless-rescue:Motor_Servo-Motor M3
 U 1 1 5CEA7A5C
 P 3200 3600
@@
 $EndComp
 $Comp
-L Device:R R19
+L EggbotWireless-rescue:R-Device R19
 U 1 1 5CECA907
 P 9100 5900
@@
 	9100 4600 9100 5200
 $Comp
-L Transistor_FET:2N7002 Q2
+L EggbotWireless-rescue:2N7002-Transistor_FET Q2
 U 1 1 5CF2F5A0
 P 8600 5850
@@
 $EndComp
 $Comp
-L power:+3.3V #PWR0135
+L EggbotWireless-rescue:+3.3V-power #PWR0135
 U 1 1 5CEC8E18
 P 9100 6050
@@
 Connection ~ 4600 5300
 $Comp
-L Driver_Motor:Pololu_Breakout_DRV8825 A2
+L EggbotWireless-rescue:Pololu_Breakout_DRV8825-Driver_Motor A2
 U 1 1 5CE8A6D5
 P 5000 5600
@@
 Connection ~ 4550 3450
 $Comp
-L Driver_Motor:Pololu_Breakout_DRV8825 A1
+L EggbotWireless-rescue:Pololu_Breakout_DRV8825-Driver_Motor A1
 U 1 1 5CE88FAE
 P 4950 3750
@@
 	4450 4350 4550 4350
 $Comp
-L power:+3.3V #PWR0146
+L EggbotWireless-rescue:+3.3V-power #PWR0146
 U 1 1 5D2FA0EE
 P 4150 4150
@@
 	4050 4350 4050 4550
 $Comp
-L power:+3.3V #PWR0138
+L EggbotWireless-rescue:+3.3V-power #PWR0138
 U 1 1 5CEA2E4D
 P 1800 4900
@@
 $EndComp
 $Comp
-L power:+3.3V #PWR0137
+L EggbotWireless-rescue:+3.3V-power #PWR0137
 U 1 1 5CEA2524
 P 1500 4900
@@
 SDA
 $Comp
-L MCU_Microchip_ATmega:ATmega328P-AU U2
+L EggbotWireless-rescue:ATmega328P-AU-MCU_Microchip_ATmega U2
 U 1 1 5D42120B
 P 1550 2550
@@
 	2500 2850 2500 2800
 $Comp
-L power:+3.3V #PWR0151
+L EggbotWireless-rescue:+3.3V-power #PWR0151
 U 1 1 5D6D37B2
 P 2500 2500
@@
 	1150 5700 2200 5700
 $Comp
-L Device:Q_NMOS_GDS Q1
+L EggbotWireless-rescue:Q_NMOS_GDS-Device Q1
 U 1 1 5CEE2D00
 P 9600 4750
@@
 $EndComp
 $Comp
-L power:+5V #PWR0102
+L EggbotWireless-rescue:+5V-power #PWR0102
 U 1 1 5D136419
 P 9100 2650
@@
 Connection ~ 9100 2650
 $Comp
-L power:+5V #PWR0108
+L EggbotWireless-rescue:+5V-power #PWR0108
 U 1 1 5D15A988
 P 9300 3800
@@
 $EndComp
 $Comp
-L power:+5V #PWR0109
+L EggbotWireless-rescue:+5V-power #PWR0109
 U 1 1 5D15FDEC
 P 2900 3600
@@
 $EndComp
 $Comp
-L Interface_USB:FT232RL U5
+L EggbotWireless-rescue:FT232RL-Interface_USB U5
 U 1 1 5D0B79CF
 P 7400 3200
@@
 	4200 1200 4300 1200
 $Comp
-L power:+12V #PWR0101
+L EggbotWireless-rescue:+12V-power #PWR0101
 U 1 1 5CEAFAB1
 P 4300 1100
@@
 $EndComp
 $Comp
-L power:+3.3V #PWR0110
+L EggbotWireless-rescue:+3.3V-power #PWR0110
 U 1 1 5CEB1C70
 P 4300 1200
@@
 $EndComp
 $Comp
-L Motor:Stepper_Motor_bipolar M1
+L EggbotWireless-rescue:Stepper_Motor_bipolar-Motor M1
 U 1 1 5CF4B0D1
 P 6000 3950
@@
 $EndComp
 $Comp
-L Motor:Stepper_Motor_bipolar M2
+L EggbotWireless-rescue:Stepper_Motor_bipolar-Motor M2
 U 1 1 5CF4C34B
 P 5950 5800
@@
 $EndComp
 $Comp
-L power:+3.3V #PWR0122
+L EggbotWireless-rescue:+3.3V-power #PWR0122
 U 1 1 5CEB99B1
 P 10900 2500
@@
 $EndComp
 $Comp
-L Device:D_Schottky D2
+L EggbotWireless-rescue:D_Schottky-Device D2
 U 1 1 5D797446
 P 10150 1950
@@
 $EndComp
 $Comp
-L Switch:SW_SPDT SW1
+L EggbotWireless-rescue:SW_SPDT-Switch SW1
 U 1 1 5CEB7C0D
 P 10750 1400
@@
 $EndComp
 $Comp
-L power:+5V #PWR0130
+L EggbotWireless-rescue:+5V-power #PWR0130
 U 1 1 5D7ABED4
 P 10950 1300
@@
 Connection ~ 8700 6200
 $Comp
-L power:+3.3V #PWR0153
+L EggbotWireless-rescue:+3.3V-power #PWR0153
 U 1 1 5D0D61D4
 P 7300 2200
@@
 SLEEP
 $Comp
-L Device:LED D3
+L EggbotWireless-rescue:LED-Device D3
 U 1 1 5D296C74
 P 4900 1200
@@
 CHEN
 $Comp
-L Device:CP C12
+L EggbotWireless-rescue:CP-Device C12
 U 1 1 5D6221F0
 P 10500 2800
@@
 GPIO0
 $Comp
-L Device:Q_NPN_BEC Q5
+L EggbotWireless-rescue:Q_NPN_BEC-Device Q5
 U 1 1 5D2B6423
 P 4500 6650
@@
 $EndComp
 $Comp
-L Device:Q_NPN_BEC Q6
+L EggbotWireless-rescue:Q_NPN_BEC-Device Q6
 U 1 1 5D2BB966
 P 4500 7350
@@
 $EndComp
 $Comp
-L Connector:Conn_01x03_Male J2
+L EggbotWireless-rescue:Conn_01x03_Male-Connector J2
 U 1 1 5D2FE20C
 P 4000 1100
@@
 $EndComp
 $Comp
-L power:+5V #PWR0111
+L EggbotWireless-rescue:+5V-power #PWR0111
 U 1 1 5D283EF7
 P 7500 2200
@@
 TXD_USB
 $Comp
-L Connector:Conn_01x05_Male J6
+L EggbotWireless-rescue:Conn_01x05_Male-Connector J6
 U 1 1 5D0DB384
 P 4000 1750
@@
 Connection ~ 5900 1950
 $Comp
-L Transistor_FET:IRLML6402 Q4
+L EggbotWireless-rescue:IRLML6402-Transistor_FET Q4
 U 1 1 5D31E4EE
 P 6100 1950
@@
 	10400 4450 10550 4450
 $Comp
-L power:+12V #PWR0124
+L EggbotWireless-rescue:+12V-power #PWR0124
 U 1 1 5CF327F6
 P 10550 4450
@@
 $EndComp
 $Comp
-L Device:D_Schottky D4
+L EggbotWireless-rescue:D_Schottky-Device D4
 U 1 1 5D32EDF7
 P 10200 650
@@
 	9050 3850 9300 3850
 $Comp
-L Device:C C17
+L EggbotWireless-rescue:C-Device C17
 U 1 1 5D338D3C
 P 9700 4000
@@
 Connection ~ 9300 4150
 $Comp
-L Transistor_FET:IRLML6402 Q3
+L EggbotWireless-rescue:IRLML6402-Transistor_FET Q3
 U 1 1 5D2DC610
 P 10250 1100
@@
 	10450 1400 10550 1400
 $Comp
-L Jumper:SolderJumper_2_Bridged JP3
+L EggbotWireless-rescue:SolderJumper_2_Bridged-Jumper JP3
 U 1 1 5D3CD55E
 P 4300 4150
@@
 $EndComp
 $Comp
-L Jumper:SolderJumper_2_Bridged JP2
+L EggbotWireless-rescue:SolderJumper_2_Bridged-Jumper JP2
 U 1 1 5D3CED16
 P 4250 4350
@@
 $EndComp
 $Comp
-L Jumper:SolderJumper_2_Bridged JP1
+L EggbotWireless-rescue:SolderJumper_2_Bridged-Jumper JP1
 U 1 1 5D3CF16C
 P 4200 4550
